File: Board/OpenParol.kicad_sch (KiCad schematic)
At the start: 242 parts, among them J1 XT30PW-M, J10 15EDGVC38108P1400AH, J11 15EDGVC38108P1400AH, J12 15EDGVC38108P1400AH, J13 15EDGVC38108P1400AH, J2 USB_C_Receptacle_USB2.0_16P, J3 Conn_01x05_Pin, J4 Conn_ARM_JTAG_SWD_10, J5 Conn_01x02_Socket, J6 15EDGVC38108P1400AH, J7 15EDGVC38108P1400AH, J8 15EDGVC38108P1400AH, J9 15EDGVC38108P1400AH, Q1 SI7157DP-T1-GE3, Q2 SI7157DP-T1-GE3, Q3 SI2310, Q4 SI2310, SW1 PTS647SN50SMTR2 LFS, SW2 PTS647SN50SMTR2 LFS, U1 LMR33630CRNXR, U10 ISO1042DWV, U11 ISO1042DWV, U12 ISO1228, U13 NSI50010YT1G, U14 TLP293, U15 NSI50010YT1G, U16 TLP293, U17 TLP3545A(TP1,F, U18 TLP3545A(TP1,F, U2 AP2114H-3.3TRG1, U3 STM32G474VET6, U4 TMC5160T, U5 TMC5160T, U6 TMC5160T, U7 TMC5160T, U8 TMC5160T, U9 TMC5160T, Y1 16MHz

Commit message: chore: rename Board to board and update schematic
Parts:
- D8: MPN SMLEN3BC8TT86 -> VAOL-S6SB4
Other:
- note removed: "TODO: Poprawić rezystor i diodę na 20mA"
- moved on the sheet: R17
